File: gateway.sch (EAGLE design)
At the start: 66 parts, among them J1 RASPBERRYPI-40-PIN-GPIO_PTH_N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, Q1 BSS123

Commit message: added a 2mm tplace line around board.
changed rain header to 1.5mm pitch
Parts:
- added C3, C4: (no value), rcl:C-USC1812
- RAIN: value JST-PH_3-PIN_HEADER -> B3B-ZR; device SRG:JST-PH_3-PIN_HEADER -> jst:B3B-ZR
Connections:
- net +5V: now also C3.1, C4.1
- net GND: now also C3.2, C4.2
Other:
- moved on the sheet: RAIN
Changed lines of the file:
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@@
 <part name="U$2" library="edc_modules" deviceset="MINI_360_BUCK" device=""/>
 <part name="RPI_VIN" library="SRG" deviceset="JST-PH_2-PIN_HEADER" device=""/>
-<part name="RAIN" library="SRG" deviceset="JST-PH_3-PIN_HEADER" device=""/>
 <part name="GND11" library="supply1" deviceset="GND" device=""/>
 <part name="BATT" library="SRG" deviceset="JST-PH_2-PIN_HEADER" device=""/>
@@
 <part name="FUSE1" library="fuse" deviceset="MF-SMDF" device="" technology="200"/>
 <part name="FUSE2" library="fuse" deviceset="MF-SMDF" device="" technology="200"/>
+<part name="C3" library="rcl" deviceset="C-US" device="C1812"/>
+<part name="C4" library="rcl" deviceset="C-US" device="C1812"/>
+<part name="RAIN" library="jst" deviceset="B3B-ZR" device=""/>
 </parts>
 <sheets>
@@
 <instance part="U$2" gate="G$1" x="213.36" y="53.34"/>
 <instance part="RPI_VIN" gate="G$1" x="226.06" y="96.52" rot="R180"/>
-<instance part="RAIN" gate="G$1" x="215.9" y="149.86" smashed="yes" rot="R180">
-<attribute name="NAME" x="218.44" y="144.018" size="1.27" layer="95" rot="R180"/>
-</instance>
 <instance part="GND11" gate="1" x="236.22" y="55.88"/>
 <instance part="BATT" gate="G$1" x="160.02" y="66.04" smashed="yes">
@@
 <instance part="FUSE1" gate="A" x="172.72" y="73.66"/>
 <instance part="FUSE2" gate="A" x="243.84" y="68.58"/>
+<instance part="C3" gate="G$1" x="309.88" y="215.9"/>
+<instance part="C4" gate="G$1" x="320.04" y="215.9"/>
+<instance part="RAIN" gate="G$1" x="246.38" y="127" rot="R180"/>
 </instances>
 <busses>
@@
 <junction x="241.3" y="142.24"/>
 <junction x="233.68" y="142.24"/>
-<pinref part="RAIN" gate="G$1" pin="1"/>
 </segment>
 <segment>
@@
 <label x="261.62" y="160.02" size="1.778" layer="95"/>
 </segment>
+<segment>
+<pinref part="C4" gate="G$1" pin="2"/>
+<wire x1="309.88" y1="210.82" x2="320.04" y2="210.82" width="0.1524" layer="91"/>
+<pinref part="C3" gate="G$1" pin="2"/>
+</segment>
+<segment>
+<pinref part="RAIN" gate="G$1" pin="1"/>
+<wire x1="254" y1="124.46" x2="264.16" y2="124.46" width="0.1524" layer="91"/>
+</segment>
 </net>
 <net name="INA_VIN-" class="0">
@@
 </segment>
 <segment>
-<wire x1="220.98" y1="149.86" x2="233.68" y2="149.86" width="0.1524" layer="91"/>
+<wire x1="220.98" y1="149.86" x2="241.3" y2="149.86" width="0.1524" layer="91"/>
 <label x="226.06" y="149.86" size="1.778" layer="95"/>
 <pinref part="C1" gate="G$1" pin="1"/>
-<wire x1="233.68" y1="149.86" x2="241.3" y2="149.86" width="0.1524" layer="91"/>
 <pinref part="C2" gate="G$1" pin="1"/>
 <wire x1="248.92" y1="149.86" x2="241.3" y2="149.86" width="0.1524" layer="91"/>
 <junction x="241.3" y="149.86"/>
+</segment>
+<segment>
 <pinref part="RAIN" gate="G$1" pin="2"/>
+<wire x1="254" y1="127" x2="264.16" y2="127" width="0.1524" layer="91"/>
 </segment>
 </net>
@@
 <pinref part="P+2" gate="1" pin="+5V"/>
 <wire x1="248.92" y1="68.58" x2="264.16" y2="68.58" width="0.1524" layer="91"/>
+</segment>
+<segment>
+<pinref part="C3" gate="G$1" pin="1"/>
+<pinref part="C4" gate="G$1" pin="1"/>
+<wire x1="309.88" y1="218.44" x2="320.04" y2="218.44" width="0.1524" layer="91"/>
 </segment>
 </net>
@@
 <wire x1="220.98" y1="152.4" x2="233.68" y2="152.4" width="0.1524" layer="91"/>
 <pinref part="+3V5" gate="G$1" pin="+3V3"/>
+</segment>
+<segment>
 <pinref part="RAIN" gate="G$1" pin="3"/>
-</segment>
-</net>
+<wire x1="254" y1="129.54" x2="264.16" y2="129.54" width="0.1524" layer="91"/>
+</segment>
+</net>

Commit message: fixed all drc errors
Connections:
- net +3V3: no longer RTC.5
- net FEATHER_3.3V: now also RTC.5
Changed lines of the file:
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@@
 <part name="GND2" library="supply1" deviceset="GND" device=""/>
 <part name="GND3" library="supply1" deviceset="GND" device=""/>
-<part name="+3V1" library="supply1" deviceset="+3V3" device=""/>
 <part name="+3V2" library="supply1" deviceset="+3V3" device=""/>
 <part name="RTC" library="pinhead" deviceset="PINHD-1X5" device=""/>
-<part name="+3V3" library="supply1" deviceset="+3V3" device=""/>
 <part name="GND4" library="supply1" deviceset="GND" device=""/>
 <part name="GND5" library="supply1" deviceset="GND" device=""/>
@@
 <part name="GND7" library="supply1" deviceset="GND" device=""/>
 <part name="GND8" library="supply1" deviceset="GND" device=""/>
-<part name="+3V5" library="supply1" deviceset="+3V3" device=""/>
 <part name="C1" library="rcl" deviceset="C-EU" device="C0805"/>
 <part name="C2" library="rcl" deviceset="C-EU" device="C0805"/>
@@
 <instance part="GND2" gate="1" x="147.32" y="154.94" rot="R270"/>
 <instance part="GND3" gate="1" x="182.88" y="101.6" rot="R90"/>
-<instance part="+3V1" gate="G$1" x="180.34" y="106.68"/>
 <instance part="+3V2" gate="G$1" x="76.2" y="119.38"/>
 <instance part="RTC" gate="A" x="193.04" y="96.52" rot="R180"/>
-<instance part="+3V3" gate="G$1" x="195.58" y="109.22"/>
 <instance part="GND4" gate="1" x="210.82" y="91.44" rot="R90"/>
 <instance part="GND5" gate="1" x="71.12" y="104.14" rot="R270"/>
@@
 <instance part="GND7" gate="1" x="71.12" y="109.22" rot="R270"/>
 <instance part="GND8" gate="1" x="233.68" y="134.62"/>
-<instance part="+3V5" gate="G$1" x="233.68" y="154.94"/>
 <instance part="C1" gate="G$1" x="241.3" y="147.32"/>
 <instance part="C2" gate="G$1" x="248.92" y="147.32"/>
@@
 <wire x1="205.74" y1="58.42" x2="208.28" y2="58.42" width="0.1524" layer="91"/>
 <pinref part="U$2" gate="G$1" pin="VIN-"/>
+<junction x="205.74" y="58.42"/>
+<junction x="208.28" y="58.42"/>
+<junction x="203.2" y="58.42"/>
 </segment>
 <segment>
@@
 <wire x1="86.36" y1="116.84" x2="76.2" y2="116.84" width="0.1524" layer="91"/>
 <pinref part="J1" gate="G$1" pin="3.3V@1"/>
-</segment>
-<segment>
-<pinref part="RTC" gate="A" pin="5"/>
-<wire x1="195.58" y1="101.6" x2="195.58" y2="106.68" width="0.1524" layer="91"/>
-<pinref part="+3V3" gate="G$1" pin="+3V3"/>
 </segment>
 </net>
@@
 <segment>
 <wire x1="162.56" y1="104.14" x2="180.34" y2="104.14" width="0.1524" layer="91"/>
-<pinref part="+3V1" gate="G$1" pin="+3V3"/>
 <pinref part="INA219" gate="G$1" pin="VCC"/>
 </segment>
 <segment>
 <wire x1="220.98" y1="152.4" x2="233.68" y2="152.4" width="0.1524" layer="91"/>
-<pinref part="+3V5" gate="G$1" pin="+3V3"/>
 </segment>
 <segment>
 <pinref part="RAIN" gate="G$1" pin="3"/>
 <wire x1="254" y1="129.54" x2="264.16" y2="129.54" width="0.1524" layer="91"/>
+</segment>
+<segment>
+<pinref part="RTC" gate="A" pin="5"/>
+<wire x1="195.58" y1="101.6" x2="195.58" y2="106.68" width="0.1524" layer="91"/>
 </segment>
 </net>
@@
 </sheet>
 </sheets>
+<errors>
+</errors>
 </schematic>
 </drawing>

Commit message: changed bno05 vin / 3.3V connection
Connections:
- net FEATHER_3.3V: now also U$4.VIN; no longer U$4.3V3
Changed lines of the file:
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@@
-</segment>
-<segment>
-<wire x1="276.86" y1="162.56" x2="266.7" y2="162.56" width="0.1524" layer="91"/>
-<pinref part="U$4" gate="G$1" pin="3V3"/>
-<label x="261.62" y="162.56" size="1.778" layer="95"/>
 </segment>
 <segment>
@@
 <wire x1="195.58" y1="101.6" x2="195.58" y2="106.68" width="0.1524" layer="91"/>
 </segment>
+<segment>
+<pinref part="U$4" gate="G$1" pin="VIN"/>
+<wire x1="276.86" y1="165.1" x2="264.16" y2="165.1" width="0.1524" layer="91"/>
+</segment>
 </net>
