File: gateway.brd (EAGLE design)
At the start: 55.9 x 64.8 mm, 20 parts

Commit message: few gateway revisions
Parts:
- added ALARM: JST-PH_3-PIN_HEADER, SRG:JST_B3B-PH_HEADER
Connections:
- new net ALARM_TRIG: ALARM.P2, PCB2.P$7
- net +5V: now also ALARM.P3
- net GND: now also ALARM.P1
Routing:
- net +5V: track 0.00 -> 50.5 mm, vias 0 -> 6
- net ALARM_TRIG: track 0.00 -> 10.6 mm
- net +3V3: track 110.3 -> 110.8 mm
- net GND: vias 12 -> 16
- added copper zone on layer 16, net +5V
Changed lines of the file:
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@@
 <setting verticaltext="up"/>
 </settings>
-<grid distance="50" unitdist="mil" unit="mil" style="lines" multiple="1" display="yes" altdistance="5" altunitdist="mil" altunit="mil"/>
+<grid distance="10" unitdist="mil" unit="mm" style="lines" multiple="1" display="yes" altdistance="5" altunitdist="mil" altunit="mil"/>
 <layers>
 <layer number="1" name="Top" color="4" fill="1" visible="yes" active="yes"/>
@@
 <dimension x1="0" y1="0" x2="55.88" y2="0" x3="27.94" y3="-5.715" textsize="1.778" layer="150"/>
 <dimension x1="0" y1="0" x2="0" y2="64.77" x3="-5.715" y3="32.385" textsize="1.778" layer="150"/>
+<dimension x1="0" y1="-0.762" x2="55.88" y2="-0.762" x3="27.94" y3="-2.54" textsize="1.016" textratio="12" layer="51"/>
+<dimension x1="-1.27" y1="0" x2="-1.27" y2="64.77" x3="-4.826" y3="32.385" textsize="1.016" textratio="12" layer="51"/>
 </plain>
 <attributes>
@@
 <attribute name="VALUE" x="1.016" y="12.065" size="0.6096" layer="27" font="vector" ratio="20" rot="R270" align="top-left"/>
 </element>
+<element name="ALARM" library="SRG" package="JST_B3B-PH_HEADER" value="JST-PH_3-PIN_HEADER" x="45.72" y="41.91" rot="R90"/>
 </elements>
 <signals>
@@
 <vertex x="53.34" y="0"/>
 </polygon>
-<polygon width="0.4064" layer="16" isolate="0.8128">
+<polygon width="0.4064" layer="16" isolate="0.8128" rank="6">
 <vertex x="0" y="4.318"/>
 <vertex x="0" y="64.77"/>
@@
 <wire x1="52.6542" y1="44.831" x2="52.6542" y2="43.25046875" width="0.4064" layer="16"/>
 <wire x1="52.6542" y1="43.25046875" x2="53.7718" y2="42.13286875" width="0.4064" layer="16"/>
-<via x="22.86" y="46.99" extent="1-16" drill="0.35"/>
-<via x="24.13" y="46.99" extent="1-16" drill="0.35"/>
-<via x="25.4" y="46.99" extent="1-16" drill="0.35"/>
-<via x="26.67" y="46.99" extent="1-16" drill="0.35"/>
-<via x="48.26" y="39.37" extent="1-16" drill="0.35"/>
-<via x="46.99" y="39.37" extent="1-16" drill="0.35"/>
-<via x="46.99" y="40.64" extent="1-16" drill="0.35"/>
-<via x="48.26" y="40.64" extent="1-16" drill="0.35"/>
+<via x="14.732" y="44.45" extent="1-16" drill="0.35"/>
+<via x="16.002" y="44.45" extent="1-16" drill="0.35"/>
+<via x="17.272" y="44.45" extent="1-16" drill="0.35"/>
+<via x="18.542" y="44.45" extent="1-16" drill="0.35"/>
+<via x="44.958" y="36.068" extent="1-16" drill="0.35"/>
+<via x="43.688" y="36.068" extent="1-16" drill="0.35"/>
+<via x="43.688" y="37.338" extent="1-16" drill="0.35"/>
+<via x="44.958" y="37.338" extent="1-16" drill="0.35"/>
 <contactref element="RFM9X_LORA" pad="2"/>
 <via x="20.32" y="17.78" extent="1-16" drill="0.35"/>
 <via x="20.32" y="19.05" extent="1-16" drill="0.35"/>
-<via x="45.72" y="40.64" extent="1-16" drill="0.35"/>
-<via x="45.72" y="39.37" extent="1-16" drill="0.35"/>
+<via x="42.418" y="37.338" extent="1-16" drill="0.35"/>
+<via x="42.418" y="36.068" extent="1-16" drill="0.35"/>
 <contactref element="BATT" pad="2"/>
 <wire x1="52.6542" y1="13.69633125" x2="53.7718" y2="14.81393125" width="0.4064" layer="1"/>
@@
 <wire x1="44.45" y1="25.4" x2="43.688" y2="26.162" width="0.4064" layer="16"/>
 <wire x1="43.688" y1="26.162" x2="43.688" y2="27.94" width="0.4064" layer="16"/>
+<contactref element="ALARM" pad="P1"/>
+<via x="32.766" y="36.322" extent="1-16" drill="0.35"/>
+<via x="34.036" y="36.322" extent="1-16" drill="0.35"/>
+<via x="35.306" y="36.322" extent="1-16" drill="0.35"/>
+<via x="36.576" y="36.322" extent="1-16" drill="0.35"/>
 </signal>
 <signal name="RPI_TX">
@@
 <wire x1="21.5138" y1="29.1338" x2="19.939" y2="29.1338" width="1.778" layer="16"/>
 <contactref element="PCB2" pad="P$17"/>
-<wire x1="51.2318" y1="36.0934" x2="45.72" y2="36.0934" width="1.778" layer="16"/>
-<wire x1="45.72" y1="36.0934" x2="40.64" y2="36.0934" width="1.778" layer="16"/>
-<wire x1="40.64" y1="36.0934" x2="28.4734" y2="36.0934" width="1.778" layer="16"/>
-<wire x1="28.4734" y1="36.0934" x2="21.5138" y2="29.1338" width="1.778" layer="16"/>
-<wire x1="46.228" y1="27.94" x2="46.228" y2="35.5854" width="1.778" layer="16"/>
-<wire x1="46.228" y1="35.5854" x2="45.72" y2="36.0934" width="1.778" layer="16"/>
+<wire x1="46.1518" y1="33.5534" x2="45.72" y2="33.5534" width="1.778" layer="16"/>
+<wire x1="45.72" y1="33.5534" x2="40.64" y2="33.5534" width="1.778" layer="16"/>
+<wire x1="40.64" y1="33.5534" x2="39.37" y2="33.5534" width="1.778" layer="16"/>
+<wire x1="25.9334" y1="33.5534" x2="21.5138" y2="29.1338" width="1.778" layer="16"/>
+<wire x1="46.228" y1="27.94" x2="46.228" y2="33.0454" width="1.778" layer="16"/>
+<wire x1="46.228" y1="33.0454" x2="45.72" y2="33.5534" width="1.778" layer="16"/>
 <wire x1="49.21" y1="58.42" x2="45.72" y2="58.42" width="1.778" layer="16"/>
 <wire x1="45.72" y1="58.42" x2="41.91" y2="58.42" width="1.778" layer="16"/>
-<wire x1="41.91" y1="58.42" x2="40.64" y2="57.15" width="1.778" layer="16"/>
-<wire x1="40.64" y1="57.15" x2="40.64" y2="36.0934" width="1.778" layer="16"/>
+<wire x1="41.91" y1="58.42" x2="39.37" y2="55.88" width="1.778" layer="16"/>
+<wire x1="39.37" y1="55.88" x2="39.37" y2="37.3634" width="1.778" layer="16"/>
 <wire x1="15.8075" y1="10.3425" x2="15.8075" y2="3.8575" width="0.8128" layer="1"/>
 <wire x1="11.3625" y1="14.7875" x2="15.8075" y2="10.3425" width="0.8128" layer="1"/>
+<wire x1="48.6918" y1="36.0934" x2="46.1518" y2="33.5534" width="1.778" layer="16"/>
+<wire x1="39.37" y1="37.3634" x2="39.37" y2="33.5534" width="1.778" layer="16"/>
+<wire x1="51.2318" y1="36.0934" x2="48.6918" y2="36.0934" width="1.778" layer="16"/>
+<wire x1="39.37" y1="33.5534" x2="25.9334" y2="33.5534" width="1.778" layer="16"/>
 </signal>
 <signal name="RPI_SDA">
@@
 <vertex x="13.97" y="52.959"/>
 <vertex x="13.97" y="54.991"/>
-<vertex x="13.716" y="55.245"/>
-<vertex x="9.525" y="55.245"/>
+<vertex x="13.462" y="55.499"/>
+<vertex x="9.525" y="55.499"/>
 <vertex x="9.525" y="60.706"/>
 <vertex x="9.271" y="60.96"/>
@@
 <vertex x="6.35" y="60.706"/>
 </polygon>
+<contactref element="ALARM" pad="P3"/>
+<wire x1="45.6725" y1="39.9375" x2="37.2785" y2="39.9375" width="1.27" layer="1"/>
+<wire x1="37.2785" y1="39.9375" x2="36.83" y2="40.386" width="1.27" layer="1"/>
+<via x="36.83" y="40.386" extent="1-16" drill="0.35"/>
+<wire x1="36.83" y1="40.386" x2="36.83" y2="45.974" width="1.27" layer="16"/>
+<wire x1="10.922" y1="47.244" x2="8.382" y2="49.784" width="1.27" layer="16"/>
+<wire x1="35.56" y1="47.244" x2="10.922" y2="47.244" width="1.27" layer="16"/>
+<wire x1="36.83" y1="45.974" x2="35.56" y2="47.244" width="1.27" layer="16"/>
+<wire x1="8.382" y1="49.784" x2="8.382" y2="55.626" width="1.27" layer="16"/>
+<via x="8.382" y="55.626" extent="1-16" drill="0.35"/>
+<polygon width="0.1524" layer="16">
+<vertex x="6.858" y="56.134"/>
+<vertex x="9.906" y="56.134"/>
+<vertex x="9.906" y="52.832"/>
+<vertex x="6.858" y="52.832"/>
+</polygon>
+<via x="7.366" y="55.626" extent="1-16" drill="0.35"/>
+<via x="9.398" y="55.626" extent="1-16" drill="0.35"/>
+<via x="7.366" y="54.61" extent="1-16" drill="0.35"/>
+<via x="7.366" y="53.594" extent="1-16" drill="0.35"/>
 </signal>
 <signal name="N$5">
@@
 <vertex x="10.16" y="62.23"/>
 <vertex x="9.906" y="61.976"/>
-<vertex x="9.906" y="56.134"/>
-<vertex x="10.16" y="55.88"/>
-<vertex x="13.716" y="55.88"/>
-<vertex x="13.97" y="56.134"/>
+<vertex x="9.906" y="56.642"/>
+<vertex x="10.16" y="56.388"/>
+<vertex x="13.716" y="56.388"/>
+<vertex x="13.97" y="56.642"/>
 <vertex x="13.97" y="58.42"/>
 <vertex x="15.875" y="58.42"/>
@@
 <wire x1="30.988" y1="27.94" x2="30.988" y2="30.48" width="0.4064" layer="1"/>
 </signal>
+<signal name="ALARM_TRIG">
+<contactref element="PCB2" pad="P$7"/>
+<contactref element="ALARM" pad="P2"/>
+<wire x1="51.2318" y1="48.7934" x2="50.6984" y2="48.26" width="0.4064" layer="1"/>
+<wire x1="50.6984" y1="48.26" x2="49.53" y2="48.26" width="0.4064" layer="1"/>
+<wire x1="49.53" y1="48.26" x2="48.26" y2="46.99" width="0.4064" layer="1"/>
+<wire x1="48.26" y1="46.99" x2="48.26" y2="43.18" width="0.4064" layer="1"/>
+<wire x1="48.26" y1="43.18" x2="47.0175" y2="41.9375" width="0.4064" layer="1"/>
+<wire x1="47.0175" y1="41.9375" x2="45.6725" y2="41.9375" width="0.4064" layer="1"/>
+</signal>
 </signals>
